Commit message: path para arquivos visuais da descrição do robô agora estão como caminho relativo

File: oni_description/oni.urdf.xacro (robot description, xacro)
@@ -56,11 +56,11 @@
             <origin xyz="0 0 0" rpy="0 0 -${pi/2}"/>
             <geometry>
-                <mesh filename="file:////home/augusto/ros2_ws_oni/src/oni_claw_gazebo/models/meshes/body_OC.dae" />
+                <mesh filename="file:///$(find oni_gazebo)/oni_description/meshes/body_OC.dae" />
             </geometry>
         </visual>
         <collision>
-            <origin xyz="0 0 0" rpy="$0 0 -${pi/2}"/>
+            <origin xyz="0 0 0" rpy="0 0 -${pi/2}"/>
             <geometry>
-                <mesh filename="file:////home/augusto/ros2_ws_oni/src/oni_claw_gazebo/models/meshes/body_OC.dae" />
+                <mesh filename="file:///$(find oni_gazebo)/oni_description/meshes/body_OC.dae" />
             </geometry>
         </collision>
@@ -80,5 +80,5 @@
         orientation_z="${pi/2}"
         mass="0.3"
-        mesh="file:////home/augusto/ros2_ws_oni/src/oni_claw_gazebo/models/meshes/fr_wheel.dae"
+        mesh="file:///$(find oni_gazebo)/oni_description/meshes/fr_wheel.dae"
     />
     <xacro:mecanum_wheel
@@ -91,5 +91,5 @@
         orientation_z="${-pi/2}"
         mass="0.3"
-        mesh="file:////home/augusto/ros2_ws_oni/src/oni_claw_gazebo/models/meshes/fl_wheel.dae"
+        mesh="file:///$(find oni_gazebo)/oni_description/meshes/fl_wheel.dae"
     />
     <xacro:mecanum_wheel
@@ -102,5 +102,5 @@
         orientation_z="${pi/2}"
         mass="0.3"
-        mesh="file:////home/augusto/ros2_ws_oni/src/oni_claw_gazebo/models/meshes/fr_wheel.dae"
+        mesh="file:///$(find oni_gazebo)/oni_description/meshes/fr_wheel.dae"
     />
     <xacro:mecanum_wheel
@@ -113,5 +113,5 @@
         orientation_z="${-pi/2}"
         mass="0.3"
-        mesh="file:////home/augusto/ros2_ws_oni/src/oni_claw_gazebo/models/meshes/fl_wheel.dae"
+        mesh="file:///$(find oni_gazebo)/oni_description/meshes/fl_wheel.dae"
     />
     <xacro:imu_sensor/>

File: oni_description/sensors/laser_sensor.urdf.xacro (robot description, xacro)
@@ -6,5 +6,5 @@
             <origin xyz="0 0 -0.025" rpy="0 0 ${M_PI/2}"/>
             <geometry>
-                <mesh filename="file:////home/augusto/ros2_ws_oni/src/oni_claw_gazebo/models/meshes/rplidar.dae"/>
+                <mesh filename="file:///$(find oni_gazebo)/oni_description/meshes/rplidar.dae"/>
             </geometry>
             <material name="green">
@@ -13,5 +13,5 @@
         </visual>
         <collision>
-            <origin xyz="0 0 -0.025" rpy="0 0 0"/>
+            <origin xyz="0.003 -0.003 -0.027" rpy="0 0 ${M_PI/2}"/>
             <geometry>
                 <cylinder radius="0.0375" length="0.05"/>
